Commit message: first commit

File: perimeter/urdf/perimeter.urdf (robot description, URDF)
Before this commit: robot perimeter, 35 links, 34 joints
Links:
- link base_link: geometry collision box size=1.2 0.5 0.3; visual mesh filename=package://perimeter/meshes/base_link.dae
Joints:
- joint up_left_d435_optical_joint: origin xyz=0 0 0 rpy=-1.570795 0.0 -1.570795 -> xyz=0.05 0.01 0.03 rpy=-1.57 -1.57 0
- joint up_right_d435_optical_joint: origin xyz=0 0 0 rpy=-1.570795 0.0 -1.570795 -> xyz=0.05 0.02 0.03 rpy=1.57 -1.57 0
